Commit message: 2017autumn

File: catkin_ws/src/duckietown_description/urdf/lab5916_map.urdf.xacro (robot description, xacro)
@@ -3,5 +3,5 @@
     <robot name="duckietown" xmlns:xacro="http://www.ros.org/wiki/xacro">
         <!--Parameters-->
-        <xacro:property name="tile_width" value="0.595"/>
+        <xacro:property name="tile_width" value="0.6"/>
         <xacro:property name="pos_0" value="0.09 0.035"/>
         <xacro:property name="pos_1" value="0.035 0.09"/>

File: catkin_ws/src/duckietown_description/urdf/lab5916_map_3bound.urdf.xacro (robot description, xacro)
@@ -3,5 +3,5 @@
     <robot name="duckietown" xmlns:xacro="http://www.ros.org/wiki/xacro">
         <!--Parameters-->
-        <xacro:property name="tile_width" value="0.595"/>
+        <xacro:property name="tile_width" value="0.6"/>
         <xacro:property name="pos_0" value="0.09 0.035"/>
         <xacro:property name="pos_1" value="0.035 0.09"/>

File: catkin_ws/src/duckietown_description/urdf/macros.urdf.xacro (robot description, xacro)
@@ -16,5 +16,5 @@
                     <origin xyz="${tile_width/2} ${tile_width/2} ${-tile_thickness/2}" rpy="0 0 ${rotation * pi/180}"/>
                     <geometry>
-                        <mesh filename="package://duckietown_description/urdf/meshes/${type}.dae" />
+                        <mesh filename="package://duckietown_description/urdf/meshes/${type}.dae" scale="1.0084 1.0084 1.0084"/>
                     </geometry>
                 </visual>
